File: dioboard2/diobd.kicad_pcb (KiCad board)
At the start: 2 copper layers, 53.3 x 15.2 mm, 9 parts, among them J1 socket_1x3, J2 Conn_01x03, J3 Conn_01x03, J4 Conn_01x03

Commit message: 2019 build season changes add year to back silk add signal/pin name text to front silk squeeze in two mounting holes
Routing:
- net (no net): vias 0 -> 2
Other:
- board text added: "+"
- board text added: "2019 season"
- board text added: "GROUND (blk)"
- board text added: "SIGNAL (white)"
Changed lines of the file:
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@@
   (general
     (thickness 1.5748)
-    (drawings 11)
-    (tracks 40)
+    (drawings 15)
+    (tracks 42)
     (zones 0)
     (modules 9)
@@
     (descr "Through hole angled pin header, 1x03, 2.54mm pitch, 6mm pin length, single row")
     (tags "Through hole angled pin header THT 1x03 2.54mm single row")
-    (fp_text reference J2 (at 0 -2.54) (layer F.SilkS)
-      (effects (font (size 1 1) (thickness 0.15)))
-    )
-    (fp_text value Conn_01x03 (at 4.385 8.89) (layer F.Fab)
+    (fp_text reference J2 (at -1.27 -2.032) (layer F.SilkS)
+      (effects (font (size 1 1) (thickness 0.15)))
+    )
+    (fp_text value Conn_01x03 (at 3.81 12.7) (layer F.Fab)
       (effects (font (size 1 1) (thickness 0.15)))
     )
@@
     (descr "Through hole straight pin header, 1x03, 2.54mm pitch, single row")
     (tags "Through hole pin header THT 1x03 2.54mm single row")
-    (fp_text reference J3 (at 0 -2.33) (layer F.SilkS)
+    (fp_text reference J3 (at -0.508 -2.286) (layer F.SilkS)
       (effects (font (size 1 1) (thickness 0.15)))
     )
@@
     )
   )
+  (gr_text "2019 season" (at 105.41 101.6) (layer B.SilkS)
+    (effects (font (size 1.5 1.5) (thickness 0.2032)) (justify mirror))
+  )
+  (gr_text "SIGNAL (white)" (at 139.7 100.965) (layer F.SilkS)
+    (effects (font (size 1.5 1.016) (thickness 0.2032)))
+  )
+  (gr_text "GROUND (blk)" (at 137.668 88.9) (layer F.SilkS)
+    (effects (font (size 1.27 1.016) (thickness 0.2032)))
+  )
+  (gr_text + (at 133.35 95.25) (layer F.SilkS)
+    (effects (font (size 1.778 1.524) (thickness 0.2032)))
+  )
   (gr_line (start 119.38 104.14) (end 120.65 101.6) (layer F.Fab) (width 0.2))
   (gr_line (start 102.87 105.41) (end 101.6 100.33) (layer F.Fab) (width 0.2))
@@
   (gr_line (start 147.32 102.87) (end 147.32 87.63) (layer Edge.Cuts) (width 0.1))
   (gr_line (start 93.98 102.87) (end 147.32 102.87) (layer Edge.Cuts) (width 0.1))
+  (via (at 144.526 89.408) (size 2.794) (drill 2.286) (layers F.Cu B.Cu) (net 0))
+  (via (at 96.266 101.092) (size 2.794) (drill 2.286) (layers F.Cu B.Cu) (net 0))
   (segment (start 102.87 93.98) (end 101.6 95.25) (width 0.254) (layer B.Cu) (net 1))
   (segment (start 110.49 93.98) (end 102.87 93.98) (width 0.254) (layer B.Cu) (net 1))
